File: Max7219_FC16.kicad_sch (KiCad schematic)
At the start: 0 parts

Commit message: so many changes.
Other:
- sheet Max7219_8x10 ports: added VUSB; removed VCC
- sheet Max7219_8x11 ports: added VUSB; removed VCC
- sheet Max7219_8x8 ports: added VUSB; removed VCC
- sheet Max7219_8x9 ports: added VUSB; removed VCC
Changed lines of the file:
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@@
 (kicad_sch (version 20230121) (generator eeschema)
   (paper "A4")
+  (junction (at 73.66 35.56) (diameter 0) (color 0 0 0 0)
+  )
+  (junction (at 118.11 35.56) (diameter 0) (color 0 0 0 0)
+  )
   (junction (at 30.48 53.34) (diameter 0) (color 0 0 0 0)
   )
@@
   (junction (at 30.48 50.8) (diameter 0) (color 0 0 0 0)
   )
-  (junction (at 73.66 39.37) (diameter 0) (color 0 0 0 0)
-  )
   (junction (at 118.11 52.07) (diameter 0) (color 0 0 0 0)
   )
   (junction (at 118.11 41.91) (diameter 0) (color 0 0 0 0)
   )
-  (junction (at 118.11 39.37) (diameter 0) (color 0 0 0 0)
+  (junction (at 30.48 35.56) (diameter 0) (color 0 0 0 0)
   )
   (junction (at 73.66 52.07) (diameter 0) (color 0 0 0 0)
@@
     (stroke (width 0) (type default))
   )
-  (wire (pts (xy 118.11 39.37) (xy 162.56 39.37))
-    (stroke (width 0) (type default))
-  )
   (wire (pts (xy 73.66 54.61) (xy 118.11 54.61))
     (stroke (width 0) (type default))
@@
     (stroke (width 0) (type default))
   )
+  (wire (pts (xy 21.59 35.56) (xy 30.48 35.56))
+    (stroke (width 0) (type default))
+  )
   (wire (pts (xy 73.66 38.1) (xy 73.66 39.37))
     (stroke (width 0) (type default))
@@
     (stroke (width 0) (type default))
   )
-  (wire (pts (xy 30.48 38.1) (xy 73.66 38.1))
-    (stroke (width 0) (type default))
-  )
   (wire (pts (xy 113.03 48.26) (xy 110.49 48.26))
     (stroke (width 0) (type default))
@@
     (stroke (width 0) (type default))
   )
+  (wire (pts (xy 118.11 35.56) (xy 162.56 35.56))
+    (stroke (width 0) (type default))
+  )
   (wire (pts (xy 73.66 53.34) (xy 73.66 54.61))
     (stroke (width 0) (type default))
@@
     (stroke (width 0) (type default))
   )
+  (wire (pts (xy 73.66 35.56) (xy 118.11 35.56))
+    (stroke (width 0) (type default))
+  )
   (wire (pts (xy 30.48 95.25) (xy 26.67 95.25))
     (stroke (width 0) (type default))
   )
-  (wire (pts (xy 73.66 39.37) (xy 118.11 39.37))
-    (stroke (width 0) (type default))
+  (wire (pts (xy 30.48 35.56) (xy 73.66 35.56))
+    (stroke (width 0) (type default))
+  )
+  (global_label "VUSB" (shape input) (at 21.59 35.56 180) (fields_autoplaced)
+    (effects (font (size 1.27 1.27)) (justify right))
+    (property "Intersheetrefs" "${INTERSHEET_REFS}" (at 13.7062 35.56 0)
+      (effects (font (size 1.27 1.27)) (justify right) hide)
+    )
   )
   (sheet (at 73.66 25.4) (size 36.83 43.18) (fields_autoplaced)
@@
       (effects (font (size 1.27 1.27)) (justify left))
     )
-    (pin "VCC" input (at 73.66 39.37 180)
-      (effects (font (size 1.27 1.27)) (justify left))
-    )
     (pin "CLK" input (at 73.66 52.07 180)
       (effects (font (size 1.27 1.27)) (justify left))
@@
       (effects (font (size 1.27 1.27)) (justify left))
     )
+    (pin "VUSB" input (at 73.66 35.56 180)
+      (effects (font (size 1.27 1.27)) (justify left))
+    )
     (instances
       (project "Max7219_FC16"
@@
       (effects (font (size 1.27 1.27)) (justify left))
     )
-    (pin "VCC" input (at 118.11 39.37 180)
-      (effects (font (size 1.27 1.27)) (justify left))
-    )
     (pin "CLK" input (at 118.11 52.07 180)
       (effects (font (size 1.27 1.27)) (justify left))
@@
       (effects (font (size 1.27 1.27)) (justify left))
     )
+    (pin "VUSB" input (at 118.11 35.56 180)
+      (effects (font (size 1.27 1.27)) (justify left))
+    )
     (instances
       (project "Max7219_FC16"
@@
       (effects (font (size 1.27 1.27)) (justify left))
     )
-    (pin "VCC" input (at 162.56 39.37 180)
-      (effects (font (size 1.27 1.27)) (justify left))
-    )
     (pin "CLK" input (at 162.56 52.07 180)
       (effects (font (size 1.27 1.27)) (justify left))
@@
       (effects (font (size 1.27 1.27)) (justify left))
     )
+    (pin "VUSB" input (at 162.56 35.56 180)
+      (effects (font (size 1.27 1.27)) (justify left))
+    )
     (instances
       (project "Max7219_FC16"
@@
       (effects (font (size 1.27 1.27)) (justify left))
     )
-    (pin "VCC" input (at 30.48 38.1 180)
-      (effects (font (size 1.27 1.27)) (justify left))
-    )
     (pin "CLK" input (at 30.48 50.8 180)
       (effects (font (size 1.27 1.27)) (justify left))
@@
       (effects (font (size 1.27 1.27)) (justify left))
     )
+    (pin "VUSB" input (at 30.48 35.56 180)
+      (effects (font (size 1.27 1.27)) (justify left))
+    )

Commit message: almost to jlpcb
Parts:
- added J2: Conn_01x05_Pin, Connector_PinHeader_2.54mm:PinHeader_1x05_P2.54mm_Vertical, symbol Connector:Conn_01x05_Pin
Connections:
- net ESP32 Section/CLK: now also J2.4 (Pin_4)
- net ESP32 Section/CS: now also J2.5 (Pin_5)
- net ESP32 Section/MOSI: now also J2.3 (Pin_3)
- net VUSB: now also J2.1 (Pin_1)
- new net GND: J2.2 (Pin_2)
Changed lines of the file:
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@@
 (kicad_sch (version 20230121) (generator eeschema)
   (paper "A4")
+  (junction (at 24.13 53.34) (diameter 0) (color 0 0 0 0)
+  )
   (junction (at 73.66 35.56) (diameter 0) (color 0 0 0 0)
   )
@@
   (junction (at 30.48 50.8) (diameter 0) (color 0 0 0 0)
   )
+  (junction (at 26.67 55.88) (diameter 0) (color 0 0 0 0)
+  )
+  (junction (at 26.67 40.64) (diameter 0) (color 0 0 0 0)
+  )
   (junction (at 118.11 52.07) (diameter 0) (color 0 0 0 0)
   )
+  (junction (at 30.48 40.64) (diameter 0) (color 0 0 0 0)
+  )
+  (junction (at 29.21 58.42) (diameter 0) (color 0 0 0 0)
+  )
   (junction (at 118.11 41.91) (diameter 0) (color 0 0 0 0)
   )
@@
     (stroke (width 0) (type default))
   )
+  (wire (pts (xy 20.32 39.37) (xy 21.59 39.37))
+    (stroke (width 0) (type default))
+  )
   (wire (pts (xy 30.48 91.44) (xy 24.13 91.44))
     (stroke (width 0) (type default))
   )
-  (wire (pts (xy 29.21 99.06) (xy 29.21 53.34))
+  (wire (pts (xy 26.67 40.64) (xy 30.48 40.64))
+    (stroke (width 0) (type default))
+  )
+  (wire (pts (xy 20.32 55.88) (xy 26.67 55.88))
+    (stroke (width 0) (type default))
+  )
+  (wire (pts (xy 29.21 58.42) (xy 29.21 53.34))
+    (stroke (width 0) (type default))
+  )
+  (wire (pts (xy 29.21 99.06) (xy 29.21 58.42))
     (stroke (width 0) (type default))
   )
@@
     (stroke (width 0) (type default))
   )
+  (wire (pts (xy 20.32 48.26) (xy 20.32 39.37))
+    (stroke (width 0) (type default))
+  )
   (wire (pts (xy 73.66 41.91) (xy 118.11 41.91))
     (stroke (width 0) (type default))
@@
     (stroke (width 0) (type default))
   )
+  (wire (pts (xy 26.67 55.88) (xy 26.67 50.8))
+    (stroke (width 0) (type default))
+  )
   (wire (pts (xy 30.48 41.91) (xy 30.48 40.64))
     (stroke (width 0) (type default))
@@
     (stroke (width 0) (type default))
   )
+  (wire (pts (xy 20.32 53.34) (xy 24.13 53.34))
+    (stroke (width 0) (type default))
+  )
   (wire (pts (xy 73.66 38.1) (xy 73.66 39.37))
     (stroke (width 0) (type default))
   )
+  (wire (pts (xy 21.59 40.64) (xy 26.67 40.64))
+    (stroke (width 0) (type default))
+  )
   (wire (pts (xy 67.31 46.99) (xy 73.66 46.99))
     (stroke (width 0) (type default))
@@
     (stroke (width 0) (type default))
   )
-  (wire (pts (xy 26.67 95.25) (xy 26.67 50.8))
+  (wire (pts (xy 26.67 95.25) (xy 26.67 55.88))
     (stroke (width 0) (type default))
   )
@@
     (stroke (width 0) (type default))
   )
+  (wire (pts (xy 24.13 53.34) (xy 24.13 48.26))
+    (stroke (width 0) (type default))
+  )
   (wire (pts (xy 73.66 53.34) (xy 73.66 54.61))
     (stroke (width 0) (type default))
@@
     (stroke (width 0) (type default))
   )
+  (wire (pts (xy 21.59 50.8) (xy 21.59 40.64))
+    (stroke (width 0) (type default))
+  )
   (wire (pts (xy 29.21 53.34) (xy 30.48 53.34))
     (stroke (width 0) (type default))
@@
     (stroke (width 0) (type default))
   )
+  (wire (pts (xy 20.32 50.8) (xy 21.59 50.8))
+    (stroke (width 0) (type default))
+  )
   (wire (pts (xy 30.48 53.34) (xy 73.66 53.34))
     (stroke (width 0) (type default))
@@
     (stroke (width 0) (type default))
   )
-  (wire (pts (xy 24.13 91.44) (xy 24.13 48.26))
+  (wire (pts (xy 24.13 91.44) (xy 24.13 53.34))
     (stroke (width 0) (type default))
   )
@@
     (stroke (width 0) (type default))
   )
+  (wire (pts (xy 26.67 41.91) (xy 26.67 40.64))
+    (stroke (width 0) (type default))
+  )
   (wire (pts (xy 118.11 49.53) (xy 113.03 49.53))
     (stroke (width 0) (type default))
@@
     (stroke (width 0) (type default))
   )
+  (wire (pts (xy 20.32 58.42) (xy 29.21 58.42))
+    (stroke (width 0) (type default))
+  )
   (wire (pts (xy 30.48 35.56) (xy 73.66 35.56))
+    (stroke (width 0) (type default))
+  )
+  (wire (pts (xy 21.59 39.37) (xy 21.59 35.56))
     (stroke (width 0) (type default))
   )
@@
     )
   )
+  (symbol (lib_id "power:GND") (at 26.67 41.91 0) (unit 1)
+    (in_bom yes) (on_board yes) (dnp no) (fields_autoplaced)
+    (property "Reference" "#PWR07" (at 26.67 48.26 0)
+      (effects (font (size 1.27 1.27)) hide)
+    )
+    (property "Value" "GND" (at 26.67 46.99 0)
+      (effects (font (size 1.27 1.27)))
+    )
+    (property "Footprint" "" (at 26.67 41.91 0)
+      (effects (font (size 1.27 1.27)) hide)
+    )
+    (property "Datasheet" "" (at 26.67 41.91 0)
+      (effects (font (size 1.27 1.27)) hide)
+    )
+    (pin "1")
+    (instances
+      (project "Max7219_FC16"
+        (path "/5a3631d1-c9a6-4e30-8ab6-c98ad3ade265"
+          (reference "#PWR07") (unit 1)
+        )
+      )
+    )
+  )
+  (symbol (lib_id "Connector:Conn_01x05_Pin") (at 15.24 53.34 0) (unit 1)
+    (in_bom yes) (on_board yes) (dnp no) (fields_autoplaced)
+    (property "Reference" "J2" (at 15.875 43.18 0)
+      (effects (font (size 1.27 1.27)))
+    )
+    (property "Value" "Conn_01x05_Pin" (at 15.875 45.72 0)
+      (effects (font (size 1.27 1.27)) hide)
+    )
+    (property "Footprint" "Connector_PinHeader_2.54mm:PinHeader_1x05_P2.54mm_Vertical" (at 15.24 53.34 0)
+      (effects (font (size 1.27 1.27)) hide)
+    )
+    (property "Datasheet" "~" (at 15.24 53.34 0)
+      (effects (font (size 1.27 1.27)) hide)
+    )
+    (pin "3")
+    (pin "2")
+    (pin "1")
+    (pin "4")
+    (pin "5")
+    (instances
+      (project "Max7219_FC16"
+        (path "/5a3631d1-c9a6-4e30-8ab6-c98ad3ade265"
+          (reference "J2") (unit 1)
+        )
+      )
+    )
+  )
