File: esp32.kicad_sch (KiCad schematic)
At the start: 7 parts, among them U10 AP2112K-3.3, U9 ESP32-C3-MINI-1

Commit message: so many changes.
Changed lines of the file:
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@@
     (stroke (width 0) (type default))
+  )
+  (global_label "VUSB" (shape input) (at 123.19 31.75 180) (fields_autoplaced)
+    (effects (font (size 1.27 1.27)) (justify right))
+    (property "Intersheetrefs" "${INTERSHEET_REFS}" (at 115.3062 31.75 0)
+      (effects (font (size 1.27 1.27)) (justify right) hide)
+    )
   )
   (hierarchical_label "MOSI" (shape input) (at 186.69 110.49 0) (fields_autoplaced)
@@
     (effects (font (size 1.27 1.27)) (justify left))
   )
-  (hierarchical_label "VUSB" (shape input) (at 123.19 31.75 180) (fields_autoplaced)
-    (effects (font (size 1.27 1.27)) (justify right))
-  )
   (hierarchical_label "CS" (shape input) (at 186.69 113.03 0) (fields_autoplaced)

Commit message: almost to jlpcb
Parts:
- added C7, C8, C9: 0.1uF, Capacitor_SMD:C_0402_1005Metric, symbol Device:C
- added J1: USB_B_Micro, Connector_USB:USB_Micro-B_Amphenol_10104110_Horizontal, symbol Connector:USB_B_Micro
- added JP1: Jumper_2_Open, Jumper:SolderJumper-2_P1.3mm_Open_Pad1.0x1.5mm, symbol Jumper:Jumper_2_Open
- added R10: 10k, Resistor_SMD:R_0402_1005Metric, symbol Device:R
- added R8, R9: 0, Resistor_SMD:R_0402_1005Metric, symbol Device:R
- C5: value 0.1 -> 0.1uF
- C6: value 10 -> 10uF
- R6: value 1k -> 10k
Connections:
- net +3.3V: now also R10.1
- net CLK: now also U9.12 (GPIO0/ADC1_CH0/XTAL_32K_P); no longer U9.20 (GPIO6)
- net CS: now also U9.16 (GPIO10); no longer U9.22 (GPIO8)
- net GND: now also C7.2, C8.2, C9.2, J1.5 (GND), J1.6 (Shield), JP1.2 (B)
- net MOSI: now also U9.6 (GPIO3/ADC1_CH3); no longer U9.21 (GPIO7)
- net VUSB: now also J1.1 (VBUS)
- net at U9.23 (GPIO9): now also JP1.1 (A)
- net at U9.26 (GPIO18/USB_D-): now also R8.1
- net at U9.27 (GPIO19/USB_D+): now also R9.1
- net at R6.2, U9.8 (EN/CHIP_PU): now also C9.1
- new net: C8.1, J1.3 (D+), R9.2
- new net: C7.1, J1.2 (D-), R8.2
- new net: R10.2, U9.22 (GPIO8)
