File: Max7219_8x8.kicad_sch (KiCad schematic)
At the start: 4 parts, among them U1 KWM-30881CVB, U2 MAX7221xWG

Commit message: so many changes.
Connections:
- net VCC renamed VUSB
Changed lines of the file:
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@@
   (junction (at 34.29 31.75) (diameter 0) (color 0 0 0 0)
-  )
-  (wire (pts (xy 22.86 46.99) (xy 20.32 46.99))
-    (stroke (width 0) (type default))
-  )
-  (wire (pts (xy 20.32 55.88) (xy 20.32 54.61))
-    (stroke (width 0) (type default))
   )
   (wire (pts (xy 35.56 69.85) (xy 44.45 69.85))
@@
     (stroke (width 0) (type default))
   )
-  (wire (pts (xy 24.13 49.53) (xy 20.32 49.53))
-    (stroke (width 0) (type default))
-  )
   (wire (pts (xy 64.77 67.31) (xy 74.93 67.31))
     (stroke (width 0) (type default))
   )
   (wire (pts (xy 39.37 72.39) (xy 39.37 73.66))
-    (stroke (width 0) (type default))
-  )
-  (wire (pts (xy 130.81 40.64) (xy 134.62 40.64))
-    (stroke (width 0) (type default))
-  )
-  (wire (pts (xy 20.32 59.69) (xy 20.32 57.15))
     (stroke (width 0) (type default))
   )
@@
     (stroke (width 0) (type default))
   )
-  (wire (pts (xy 130.81 45.72) (xy 134.62 45.72))
-    (stroke (width 0) (type default))
-  )
   (wire (pts (xy 41.91 31.75) (xy 44.45 31.75))
     (stroke (width 0) (type default))
@@
     (stroke (width 0) (type default))
   )
-  (wire (pts (xy 24.13 52.07) (xy 20.32 52.07))
-    (stroke (width 0) (type default))
-  )
   (wire (pts (xy 78.74 59.69) (xy 78.74 64.77))
     (stroke (width 0) (type default))
@@
     (stroke (width 0) (type default))
   )
-  (wire (pts (xy 22.86 44.45) (xy 22.86 46.99))
-    (stroke (width 0) (type default))
-  )
   (wire (pts (xy 66.04 81.28) (xy 66.04 72.39))
     (stroke (width 0) (type default))
   )
   (wire (pts (xy 80.01 62.23) (xy 83.82 62.23))
-    (stroke (width 0) (type default))
-  )
-  (wire (pts (xy 130.81 43.18) (xy 134.62 43.18))
     (stroke (width 0) (type default))
   )
@@
     (stroke (width 0) (type default))
   )
-  (wire (pts (xy 22.86 55.88) (xy 20.32 55.88))
-    (stroke (width 0) (type default))
-  )
-  (wire (pts (xy 130.81 50.8) (xy 133.35 50.8))
-    (stroke (width 0) (type default))
-  )
   (wire (pts (xy 64.77 49.53) (xy 88.9 49.53))
     (stroke (width 0) (type default))
@@
     (stroke (width 0) (type default))
   )
-  (wire (pts (xy 22.86 59.69) (xy 20.32 59.69))
-    (stroke (width 0) (type default))
-  )
   (wire (pts (xy 34.29 31.75) (xy 34.29 26.67))
     (stroke (width 0) (type default))
@@
     (stroke (width 0) (type default))
   )
-  (wire (pts (xy 25.4 44.45) (xy 22.86 44.45))
-    (stroke (width 0) (type default))
-  )
   (wire (pts (xy 54.61 77.47) (xy 54.61 80.01))
     (stroke (width 0) (type default))
   )
   (wire (pts (xy 115.57 46.99) (xy 64.77 46.99))
-    (stroke (width 0) (type default))
-  )
-  (wire (pts (xy 130.81 48.26) (xy 133.35 48.26))
     (stroke (width 0) (type default))
   )
@@
     (stroke (width 0) (type default))
   )
-  (hierarchical_label "VCC" (shape input) (at 134.62 40.64 0) (fields_autoplaced)
-    (effects (font (size 1.27 1.27)) (justify left))
-  )
-  (hierarchical_label "CS" (shape input) (at 133.35 48.26 0) (fields_autoplaced)
-    (effects (font (size 1.27 1.27)) (justify left))
-  )
-  (hierarchical_label "VCC" (shape input) (at 54.61 26.67 90) (fields_autoplaced)
-    (effects (font (size 1.27 1.27)) (justify left))
-  )
-  (hierarchical_label "CLK" (shape input) (at 22.86 59.69 0) (fields_autoplaced)
+  (hierarchical_label "VUSB" (shape input) (at 54.61 26.67 90) (fields_autoplaced)
     (effects (font (size 1.27 1.27)) (justify left))
   )
@@
     (effects (font (size 1.27 1.27)) (justify right))
   )
-  (hierarchical_label "DOUT" (shape output) (at 134.62 45.72 0) (fields_autoplaced)
-    (effects (font (size 1.27 1.27)) (justify left))
-  )
-  (hierarchical_label "DIN" (shape input) (at 24.13 52.07 0) (fields_autoplaced)
-    (effects (font (size 1.27 1.27)) (justify left))
-  )
-  (hierarchical_label "GND" (shape input) (at 134.62 43.18 0) (fields_autoplaced)
-    (effects (font (size 1.27 1.27)) (justify left))
-  )
-  (hierarchical_label "CLK" (shape input) (at 133.35 50.8 0) (fields_autoplaced)
-    (effects (font (size 1.27 1.27)) (justify left))
-  )
   (hierarchical_label "DIN" (shape input) (at 33.02 73.66 180) (fields_autoplaced)
     (effects (font (size 1.27 1.27)) (justify right))
-  )
-  (hierarchical_label "VCC" (shape input) (at 25.4 44.45 0) (fields_autoplaced)
-    (effects (font (size 1.27 1.27)) (justify left))
-  )
-  (hierarchical_label "GND" (shape input) (at 24.13 49.53 0) (fields_autoplaced)
-    (effects (font (size 1.27 1.27)) (justify left))
   )
   (hierarchical_label "CS" (shape input) (at 35.56 66.04 180) (fields_autoplaced)
     (effects (font (size 1.27 1.27)) (justify right))
   )
-  (hierarchical_label "CS" (shape input) (at 22.86 55.88 0) (fields_autoplaced)
-    (effects (font (size 1.27 1.27)) (justify left))
-  )
   (hierarchical_label "CLK" (shape input) (at 35.56 69.85 180) (fields_autoplaced)

Commit message: machine pin headers
Parts:
- added J3, J7: Conn_01x08_Socket, Connector_PinSocket_2.54mm:PinSocket_1x08_P2.54mm_Vertical, symbol Connector:Conn_01x08_Socket
Changed lines of the file:
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@@
+    )
+  )
+  (symbol (lib_id "Connector:Conn_01x08_Socket") (at 154.94 52.07 270) (unit 1)
+    (in_bom yes) (on_board yes) (dnp no) (fields_autoplaced)
+    (property "Reference" "J3" (at 153.67 54.61 90)
+      (effects (font (size 1.27 1.27)))
+    )
+    (property "Value" "Conn_01x08_Socket" (at 153.67 57.15 90)
+      (effects (font (size 1.27 1.27)))
+    )
+    (property "Footprint" "Connector_PinSocket_2.54mm:PinSocket_1x08_P2.54mm_Vertical" (at 154.94 52.07 0)
+      (effects (font (size 1.27 1.27)) hide)
+    )
+    (property "Datasheet" "~" (at 154.94 52.07 0)
+      (effects (font (size 1.27 1.27)) hide)
+    )
+    (pin "1")
+    (pin "7")
+    (pin "8")
+    (pin "6")
+    (pin "5")
+    (pin "2")
+    (pin "4")
+    (pin "3")
+    (instances
+      (project "Max7219_FC16"
+        (path "/5a3631d1-c9a6-4e30-8ab6-c98ad3ade265/aa78cd51-fb28-420d-a0c0-b0096458006b"
+          (reference "J3") (unit 1)
+        )
+        (path "/5a3631d1-c9a6-4e30-8ab6-c98ad3ade265/54d6c786-7952-437d-8986-68fa7866a4dd"
+          (reference "J4") (unit 1)
+        )
+        (path "/5a3631d1-c9a6-4e30-8ab6-c98ad3ade265/633f3b8b-b370-4c30-8839-417c094daef8"
+          (reference "J5") (unit 1)
+        )
+        (path "/5a3631d1-c9a6-4e30-8ab6-c98ad3ade265/a25a12df-9204-4310-a2ab-e55462080266"
+          (reference "J6") (unit 1)
+        )
+      )
     )
   )
@@
         )
       )
+    )
+  )
+  (symbol (lib_id "Connector:Conn_01x08_Socket") (at 152.4 67.31 90) (unit 1)
+    (in_bom yes) (on_board yes) (dnp no) (fields_autoplaced)
+    (property "Reference" "J7" (at 153.67 62.23 90)
+      (effects (font (size 1.27 1.27)))
+    )
+    (property "Value" "Conn_01x08_Socket" (at 153.67 64.77 90)
+      (effects (font (size 1.27 1.27)))
+    )
+    (property "Footprint" "Connector_PinSocket_2.54mm:PinSocket_1x08_P2.54mm_Vertical" (at 152.4 67.31 0)
+      (effects (font (size 1.27 1.27)) hide)
+    )
+    (property "Datasheet" "~" (at 152.4 67.31 0)
+      (effects (font (size 1.27 1.27)) hide)
+    )
+    (pin "1")
+    (pin "7")
+    (pin "8")
+    (pin "6")
+    (pin "5")
+    (pin "2")
+    (pin "4")
+    (pin "3")
+    (instances
+      (project "Max7219_FC16"
+        (path "/5a3631d1-c9a6-4e30-8ab6-c98ad3ade265/aa78cd51-fb28-420d-a0c0-b0096458006b"
+          (reference "J7") (unit 1)
+        )
+        (path "/5a3631d1-c9a6-4e30-8ab6-c98ad3ade265/54d6c786-7952-437d-8986-68fa7866a4dd"
+          (reference "J8") (unit 1)
+        )
+        (path "/5a3631d1-c9a6-4e30-8ab6-c98ad3ade265/633f3b8b-b370-4c30-8839-417c094daef8"
+          (reference "J9") (unit 1)
+        )
+        (path "/5a3631d1-c9a6-4e30-8ab6-c98ad3ade265/a25a12df-9204-4310-a2ab-e55462080266"
+          (reference "J10") (unit 1)
+        )
+      )
