File: Max7219_FC16.kicad_pcb (KiCad board)
At the start: 2 copper layers, 129 x 32 mm, 23 parts, among them U1 MAX7221xWG, U10 3.3v, U2 KWM-30881CVB, U3 MAX7221xWG, U4 KWM-30881CVB, U5 MAX7221xWG, U6 KWM-30881CVB, U7 MAX7221xWG, U8 KWM-30881CVB, U9 ESP32-C3-MINI-1

Commit message: update
Parts:
- U10: value 3.3v -> AP2112K-3.3
Routing:
- net Net-(U3-DIG_4): track 9.10 -> 11.1 mm, vias 0 -> 1
- net Net-(U3-SEG_D): track 32.5 -> 31.0 mm
- net Net-(U3-SEG_A): track 38.3 -> 37.0 mm

Commit message: so many changes.
Parts:
- C1, R1: moved to F.Cu
- C5, C6, R6, R7, U10: moved to B.Cu
- moved C2 22.1 mm to (94.4, 53.0), turned to -90 degrees
- moved R2 18.2 mm to (92.7, 53.0), turned to -90 degrees
- moved C1 12.6 mm to (70.6, 52.7), turned to -90 degrees
- moved R1 11.0 mm to (69.2, 52.7)
- moved R7 10.1 mm to (43.3, 44.8), turned to -90 degrees
- moved U1 9.15 mm to (85.6, 53.0), turned to 0 degrees
- moved R5 9.07 mm to (47.3, 46.6), turned to -90 degrees
- moved R6 7.43 mm to (49.8, 46.6), turned to -90 degrees
- moved U10 6.83 mm to (40.4, 44.2), turned to 180 degrees
- moved R4 5.78 mm to (135.7, 59.0), turned to 180 degrees
- moved C3 5.63 mm to (111.3, 58.9), turned to 0 degrees
- moved U7 5.56 mm to (135.6, 52.0)
- moved C5 4.19 mm to (37.3, 43.3), turned to 0 degrees
- moved U3 3.66 mm to (61.7, 53.0)
- moved R3 2.34 mm to (108.9, 58.9), turned to 180 degrees
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Connections:
- C1 pad 1: /Max7219_8x10/VCC -> VUSB
- C2 pad 1: /Max7219_8x10/VCC -> VUSB
- C3 pad 1: /Max7219_8x10/VCC -> VUSB
- C4 pad 1: /Max7219_8x10/VCC -> VUSB
- R1 pad 1: /Max7219_8x10/VCC -> VUSB
- R2 pad 1: /Max7219_8x10/VCC -> VUSB
- R3 pad 1: /Max7219_8x10/VCC -> VUSB
- R4 pad 1: /Max7219_8x10/VCC -> VUSB
- R7 pad 1: /ESP32 Section/VUSB -> VUSB
- U1 pad 19: /Max7219_8x10/VCC -> VUSB
- U10 pad 1: /ESP32 Section/VUSB -> VUSB
- U3 pad 19: /Max7219_8x10/VCC -> VUSB
- U5 pad 19: /Max7219_8x10/VCC -> VUSB
- U7 pad 19: /Max7219_8x10/VCC -> VUSB
Routing:
- net /Max7219_8x10/VCC: track 157.8 -> 0.00 mm, vias 6 -> 0
- net VUSB: track 0.00 -> 119.9 mm, vias 0 -> 5
- net /Max7219_8x10/GND: track 188.6 -> 109.1 mm, vias 22 -> 8
- net /ESP32 Section/CLK: track 30.3 -> 96.0 mm
- net /ESP32 Section/CS: track 35.3 -> 97.3 mm
- net /Max7219_8x10/DIN: track 0.00 -> 41.2 mm
- net /Max7219_8x10/DOUT: track 0.00 -> 34.2 mm, vias 0 -> 2
- net GND: track 40.7 -> 74.2 mm, vias 1 -> 0
- net Net-(U1-SEG_C): track 13.8 -> 42.9 mm, vias 0 -> 2
- net Net-(U1-SEG_E): track 12.7 -> 39.0 mm, vias 0 -> 2
- net Net-(U7-DIG_3): track 0.00 -> 25.6 mm, vias 0 -> 2
- net Net-(U1-DIG_1): track 32.5 -> 8.55 mm, vias 0 -> 1
- net /Max7219_8x8/DOUT: track 38.5 -> 14.6 mm
- net Net-(U1-SEG_DP): track 9.13 -> 32.8 mm, vias 0 -> 2
- net Net-(U5-DIG_3): track 0.00 -> 21.0 mm, vias 0 -> 1
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
Commit message: almost to jlpcb
Parts:
- added C7: 0.1uF, Capacitor_SMD:C_0402_1005Metric, B.Cu at (45.5, 62.3)
- added C8: 0.1uF, Capacitor_SMD:C_0402_1005Metric, B.Cu at (40.8, 63.0)
- added C9: 0.1uF, Capacitor_SMD:C_0402_1005Metric, B.Cu at (48.6, 47.7)
- added J1: USB_B_Micro, Connector_USB:USB_Micro-B_Amphenol_10104110_Horizontal, B.Cu at (155.1, 53.0)
- added J2: Conn_01x05_Pin, Connector_PinHeader_2.54mm:PinHeader_1x05_P2.54mm_Vertical, F.Cu at (51.3, 48.3)
- added JP1: Jumper_2_Open, Jumper:SolderJumper-2_P1.3mm_Open_Pad1.0x1.5mm, B.Cu at (48.0, 60.1)
- added R10: 10k, Resistor_SMD:R_0402_1005Metric, B.Cu at (48.7, 57.3)
- added R8: 0, Resistor_SMD:R_0402_1005Metric, B.Cu at (43.6, 62.5)
- added R9: 0, Resistor_SMD:R_0402_1005Metric, B.Cu at (42.6, 62.5)
- C5: value 0.1 -> 0.1uF
- C6: value 10 -> 10uF
- R6: value 1k -> 10k
- moved U9 0.80 mm to (37.6, 54.6)
Connections:
- C1 pad 2: /Max7219_8x10/GND -> GND
- C2 pad 2: /Max7219_8x10/GND -> GND
- C3 pad 2: /Max7219_8x10/GND -> GND
- C4 pad 2: /Max7219_8x10/GND -> GND
- U1 pad 4: /Max7219_8x10/GND -> GND
- U1 pad 9: /Max7219_8x10/GND -> GND
- U3 pad 4: /Max7219_8x10/GND -> GND
- U3 pad 9: /Max7219_8x10/GND -> GND
- U5 pad 4: /Max7219_8x10/GND -> GND
- U5 pad 9: /Max7219_8x10/GND -> GND
- U7 pad 4: /Max7219_8x10/GND -> GND
- U7 pad 9: /Max7219_8x10/GND -> GND
- U9 pad 12: unconnected-(U9-GPIO0/ADC1_CH0/XTAL_32K_P-Pad12) -> /ESP32 Section/CLK
- U9 pad 13: unconnected-(U9-GPIO1/ADC1_CH1/XTAL_32K_N-Pad13) -> GND
- U9 pad 16: unconnected-(U9-GPIO10-Pad16) -> /ESP32 Section/CS
- U9 pad 20: /ESP32 Section/CLK -> unconnected-(U9-GPIO6-Pad20)
- U9 pad 21: /ESP32 Section/MOSI -> unconnected-(U9-GPIO7-Pad21)
- U9 pad 22: /ESP32 Section/CS -> Net-(U9-GPIO8)
- U9 pad 23: unconnected-(U9-GPIO9-Pad23) -> Net-(JP1-A)
- U9 pad 26: unconnected-(U9-GPIO18/USB_D--Pad26) -> Net-(U9-GPIO18/USB_D-)
- U9 pad 27: unconnected-(U9-GPIO19/USB_D+-Pad27) -> Net-(U9-GPIO19/USB_D+)
- U9 pad 6: unconnected-(U9-GPIO3/ADC1_CH3-Pad6) -> /ESP32 Section/MOSI
Routing:
- net GND: track 74.2 -> 206.9 mm, vias 0 -> 9
- net Net-(J1-D-): track 0.00 -> 131.6 mm
- net Net-(J1-D+): track 0.00 -> 131.3 mm
- net /Max7219_8x10/GND: track 109.1 -> 0.00 mm, vias 8 -> 0
- net VUSB: track 119.9 -> 160.2 mm, vias 5 -> 8
- net +3.3V: track 18.2 -> 30.4 mm, vias 0 -> 2
- net /ESP32 Section/MOSI: track 20.8 -> 28.3 mm, vias 3 -> 2
- net /ESP32 Section/CS: track 97.3 -> 102.2 mm
- net Net-(U9-GPIO8): track 0.00 -> 3.48 mm
- net Net-(JP1-A): track 0.00 -> 3.05 mm
- net Net-(U5-DIG_0): track 47.1 -> 44.9 mm
- net Net-(U7-DIG_1): track 37.7 -> 35.9 mm
- net Net-(U9-GPIO2/ADC1_CH2): track 9.03 -> 10.6 mm
- net Net-(U9-GPIO18/USB_D-): track 0.00 -> 1.57 mm
- net Net-(U9-GPIO19/USB_D+): track 0.00 -> 1.53 mm
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- added copper zone on B.Cu, net GND
- added copper zone on F.Cu, net GND
- removed copper zone on B.Cu, net /Max7219_8x10/GND
- removed copper zone on F.Cu, net /Max7219_8x10/GND

Commit message: machine pin headers
Parts:
- added J10: Conn_01x08_Socket, Connector_PinSocket_2.54mm:PinSocket_1x08_P2.54mm_Vertical, F.Cu at (150.8, 65.0)
- added J3: Conn_01x08_Socket, Connector_PinSocket_2.54mm:PinSocket_1x08_P2.54mm_Vertical, F.Cu at (53.8, 41.0)
- added J4: Conn_01x08_Socket, Connector_PinSocket_2.54mm:PinSocket_1x08_P2.54mm_Vertical, F.Cu at (53.9, 65.0)
- added J5: Conn_01x08_Socket, Connector_PinSocket_2.54mm:PinSocket_1x08_P2.54mm_Vertical, F.Cu at (86.2, 41.0)
- added J6: Conn_01x08_Socket, Connector_PinSocket_2.54mm:PinSocket_1x08_P2.54mm_Vertical, F.Cu at (86.2, 65.0)
- added J7: Conn_01x08_Socket, Connector_PinSocket_2.54mm:PinSocket_1x08_P2.54mm_Vertical, F.Cu at (118.5, 65.0)
- added J8: Conn_01x08_Socket, Connector_PinSocket_2.54mm:PinSocket_1x08_P2.54mm_Vertical, F.Cu at (118.5, 41.0)
- added J9: Conn_01x08_Socket, Connector_PinSocket_2.54mm:PinSocket_1x08_P2.54mm_Vertical, F.Cu at (150.8, 41.0)
- J2: moved to B.Cu
- turned J2 to 180 degrees
Connections:
- U9 pad 13: GND -> unconnected-(U9-GPIO1/ADC1_CH1/XTAL_32K_N-Pad13)
Routing:
- net GND: track 206.9 -> 218.3 mm

Commit message: latest change
Other:
- outline, holes or cut-outs redrawn
- board text added: "${CURRENT_DATE}"
- board text added: "GeneralTron Jumbo v0"
Changed lines of the file:
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@@
         (effects (font (size 1 1) (thickness 0.15)))
     )
-    (fp_text value "Conn_01x08_Socket" (at 0 20.55 90) (layer "F.Fab")
+    (fp_text value "Conn_01x08_Socket" (at 0 20.55 90) (layer "F.Fab") hide
         (effects (font (size 1 1) (thickness 0.15)))
     )
@@
         (effects (font (size 1 1) (thickness 0.15)))
     )
-    (fp_text value "Conn_01x08_Socket" (at 0 20.55 90) (layer "F.Fab")
+    (fp_text value "Conn_01x08_Socket" (at 0 20.55 90) (layer "F.Fab") hide
         (effects (font (size 1 1) (thickness 0.15)))
     )
@@
         (effects (font (size 1 1) (thickness 0.15)))
     )
-    (fp_text value "Conn_01x08_Socket" (at 0 20.55 90) (layer "F.Fab")
+    (fp_text value "Conn_01x08_Socket" (at 0 20.55 90) (layer "F.Fab") hide
         (effects (font (size 1 1) (thickness 0.15)))
     )
@@
         (effects (font (size 1 1) (thickness 0.15)))
     )
-    (fp_text value "Conn_01x08_Socket" (at 0 20.55 90) (layer "F.Fab")
+    (fp_text value "Conn_01x08_Socket" (at 0 20.55 90) (layer "F.Fab") hide
         (effects (font (size 1 1) (thickness 0.15)))
     )
@@
         (effects (font (size 1 1) (thickness 0.15)))
     )
-    (fp_text value "Conn_01x08_Socket" (at 0 20.55 90) (layer "F.Fab")
+    (fp_text value "Conn_01x08_Socket" (at 0 20.55 90) (layer "F.Fab") hide
         (effects (font (size 1 1) (thickness 0.15)))
     )
@@
         (effects (font (size 1 1) (thickness 0.15)))
     )
-    (fp_text value "Conn_01x08_Socket" (at 0 20.55 90) (layer "F.Fab")
+    (fp_text value "Conn_01x08_Socket" (at 0 20.55 90) (layer "F.Fab") hide
         (effects (font (size 1 1) (thickness 0.15)))
     )
@@
         (effects (font (size 1 1) (thickness 0.15)))
     )
-    (fp_text value "Conn_01x08_Socket" (at 0 20.55 90) (layer "F.Fab")
+    (fp_text value "Conn_01x08_Socket" (at 0 20.55 90) (layer "F.Fab") hide
         (effects (font (size 1 1) (thickness 0.15)))
     )
@@
         (effects (font (size 1 1) (thickness 0.15)))
     )
-    (fp_text value "Conn_01x08_Socket" (at 0 20.55 90) (layer "F.Fab")
+    (fp_text value "Conn_01x08_Socket" (at 0 20.55 90) (layer "F.Fab") hide
         (effects (font (size 1 1) (thickness 0.15)))
     )
@@
     )
   )
-  (gr_rect (start 28.75 37) (end 157.75 69)
-    (stroke (width 0.1) (type default)) (fill none) (layer "Edge.Cuts"))
+  (gr_line (start 34.4424 46.4312) (end 28.7528 46.4312)
+    (stroke (width 0.1) (type default)) (layer "Edge.Cuts"))
+  (gr_line (start 34.5186 62.4332) (end 34.4424 46.4312)
+    (stroke (width 0.1) (type default)) (layer "Edge.Cuts"))
+  (gr_line (start 157.75 69) (end 28.75 69)
+    (stroke (width 0.1) (type default)) (layer "Edge.Cuts"))
+  (gr_line (start 28.75 37) (end 157.75 37)
+    (stroke (width 0.1) (type default)) (layer "Edge.Cuts"))
+  (gr_line (start 157.75 37) (end 157.75 69)
+    (stroke (width 0.1) (type default)) (layer "Edge.Cuts"))
+  (gr_line (start 34.5186 62.4332) (end 28.7528 62.4332)
+    (stroke (width 0.1) (type default)) (layer "Edge.Cuts"))
+  (gr_line (start 28.7528 46.4312) (end 28.75 37)
+    (stroke (width 0.1) (type default)) (layer "Edge.Cuts"))
+  (gr_line (start 28.7528 62.4332) (end 28.75 69)
+    (stroke (width 0.1) (type default)) (layer "Edge.Cuts"))
+  (gr_text "${CURRENT_DATE}" (at 127.9398 39.3192) (layer "F.SilkS")
+    (effects (font (size 1.5 1.5) (thickness 0.3) bold) (justify left bottom))
+  )
+  (gr_text "GeneralTron Jumbo v0" (at 97.3836 39.1414) (layer "F.SilkS")
+    (effects (font (size 1.5 1.5) (thickness 0.3) bold) (justify left bottom))
+  )
   (segment (start 48.642 43.3578) (end 46.27 40.9858) (width 0.25) (layer "F.Cu") (net 1))
   (segment (start 69.1994 56.175) (end 66.3956 56.175) (width 0.25) (layer "F.Cu") (net 1))

Commit message: first max routed
Parts:
- C5, C6, C7, C8, C9, J1, J2, JP1, R10, R5, R6, R7, R8, R9, U10, U9: moved to F.Cu
- J10, J3, J4, J5, J6, J7, J8, J9, U2, U4, U6, U8: moved to B.Cu
- moved C5 36.2 mm to (7.13, 63.2)
- moved C8 35.9 mm to (10.6, 43.5)
- moved R8 35.4 mm to (13.5, 44.0), turned to 90 degrees
- moved R9 35.4 mm to (12.5, 44.0), turned to 90 degrees
- moved U10 35.2 mm to (10.2, 62.3)
- moved C7 35.2 mm to (15.3, 44.2)
- moved C6 34.9 mm to (7.18, 62.0)
- moved R7 34.6 mm to (13.1, 61.7), turned to 90 degrees
- moved JP1 33.1 mm to (17.8, 46.5), turned to 90 degrees
- moved R6 33.0 mm to (19.6, 59.9), turned to 90 degrees
- moved R5 33.0 mm to (17.2, 59.9), turned to 90 degrees
- moved C9 32.1 mm to (18.5, 58.8), turned to 90 degrees
- moved J2 31.7 mm to (21.1, 58.2)
- moved R10 31.2 mm to (18.5, 49.2), turned to 90 degrees
- moved J3 19.5 mm to (36.2, 32.7)
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Routing:
- net GND: track 218.3 -> 0.00 mm, vias 9 -> 0
- net VUSB: track 160.2 -> 0.00 mm, vias 8 -> 0
- net Net-(J1-D-): track 131.6 -> 0.00 mm
- net Net-(J1-D+): track 131.3 -> 0.00 mm
- net /ESP32 Section/CS: track 102.2 -> 0.00 mm, vias 3 -> 0
- net /ESP32 Section/CLK: track 96.7 -> 0.00 mm, vias 2 -> 0
- net Net-(U5-DIG_0): track 45.3 -> 0.00 mm, vias 2 -> 0
- net Net-(U1-SEG_C): track 42.3 -> 0.00 mm, vias 2 -> 0
- net /Max7219_8x10/DIN: track 41.2 -> 0.00 mm
- net Net-(U1-SEG_E): track 38.7 -> 0.00 mm, vias 2 -> 0
- net Net-(U7-DIG_0): track 36.4 -> 0.00 mm, vias 2 -> 0
- net Net-(U7-DIG_1): track 35.9 -> 0.00 mm, vias 2 -> 0
- net /Max7219_8x10/DOUT: track 34.2 -> 0.00 mm, vias 2 -> 0
- net Net-(U1-SEG_DP): track 32.3 -> 0.00 mm, vias 2 -> 0
- net Net-(U1-SEG_D): track 31.8 -> 0.00 mm, vias 2 -> 0
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Other:
- outline, holes or cut-outs redrawn

Commit message: update
Parts:
- JP1: value Jumper_2_Open -> Boot
- moved C5 43.2 mm to (49.5, 54.7), turned to 180 degrees
- moved C6 42.8 mm to (49.5, 55.9), turned to 180 degrees
- moved R7 40.1 mm to (53.2, 59.7), turned to 180 degrees
- moved U10 39.8 mm to (49.9, 59.0), turned to -90 degrees
- moved J2 32.5 mm to (53.7, 57.1)
- moved C8 30.6 mm to (41.2, 43.5), turned to -90 degrees
- moved JP1 30.0 mm to (47.8, 46.1), turned to 180 degrees
- moved R8 29.9 mm to (43.4, 43.6)
- moved R9 29.9 mm to (42.4, 43.6)
- moved C7 29.2 mm to (44.5, 43.5), turned to -90 degrees
- moved R10 28.5 mm to (47.0, 48.3), turned to 180 degrees
- moved C9 25.2 mm to (43.6, 58.8), turned to 0 degrees
- moved R6 22.1 mm to (41.7, 59.3)
- moved R5 21.4 mm to (38.5, 58.9), turned to 0 degrees
- moved R4 12.9 mm to (147.1, 53.0), turned to -90 degrees
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Routing:
- net GND: track 0.00 -> 211.8 mm, vias 0 -> 11
- net VUSB: track 0.00 -> 198.9 mm
- net Net-(J1-D+): track 0.00 -> 130.2 mm
- net Net-(J1-D-): track 0.00 -> 128.1 mm
- net /ESP32 Section/CLK: track 0.00 -> 113.9 mm
- net /ESP32 Section/CS: track 0.00 -> 104.8 mm
- net Net-(U1-SEG_DP): track 0.00 -> 40.0 mm, vias 0 -> 2
- net /ESP32 Section/MOSI: track 0.00 -> 39.3 mm, vias 0 -> 4
- net Net-(U1-SEG_B): track 0.00 -> 38.4 mm, vias 0 -> 2
- net +3.3V: track 0.00 -> 37.9 mm, vias 0 -> 5
- net Net-(U1-SEG_G): track 0.00 -> 34.5 mm, vias 0 -> 2
- net Net-(U1-SEG_A): track 0.00 -> 33.8 mm, vias 0 -> 2
- net Net-(U1-SEG_F): track 0.00 -> 32.2 mm, vias 0 -> 2
- net Net-(U5-SEG_A): track 0.00 -> 31.5 mm, vias 0 -> 2
- net Net-(U1-SEG_C): track 0.00 -> 27.8 mm, vias 0 -> 2
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Other:
- outline, holes or cut-outs redrawn
